File: Tracer_ECU.kicad_sch (KiCad schematic)
At the start: 148 parts, among them IC1 R5F566TEADFM#30, IC2 MPU-6500, IC3 DRV8300DPWR, IC4 DRV8300DPWR, J1 BAT, J10 ENC2, J11 ENC2_SPI, J12 LCD, J13 SDC, J14 FAN, J15 ENC1_SPI, J2 DBG, J3 TSL1401, J4 MSENS1, J5 MOT1, J6 LIGHIT, J7 MSENS2, J8 MOT2, J9 ENC1, Q1 TJ8S06M3L(T6L1,NQ), Q2 FDS6898A, Q3 FDS6898A, Q4 FDS6898A, Q5 IRLML6344TRPBF, Q6 IRLML6344TRPBF, Q7 FDS6898A, Q8 FDS6898A, Q9 FDS6898A, SW1 SW_SPDT, SW2 SW_Push, SW4 SW_Push, SW5 SW_Push, U1 NJM2732, U2 AZ1117-3.3, Y1 CSTNE20M

Commit message: RX72T追加 周辺回路作成中．
Parts:
- added C35: 0.1u, Capacitor_SMD:C_0603_1608Metric_Pad1.08x0.95mm_HandSolder, symbol Device:C_Small
- added IC5: R5F572TFADFP#30, QFP50P1600X1600X170-100N, symbol SamacSys_Parts:R5F572TFADFP#30
Connections:
- net AN000: now also IC5.90 (P40)
- net AN001: now also IC5.89 (P41)
- net AN002: now also IC5.88 (P42)
- net AN100: now also IC5.85 (P44)
- net AN101: now also IC5.84 (P45)
- net AN200: now also IC5.81 (P52)
- net EMLE: now also IC5.2 (EMLE); no longer IC1.1 (EMLE)
- net GND: now also C35.2, IC5.12 (VSS_2), IC5.3 (VSS_1), IC5.31 (VSS_3), IC5.44 (VSS_4), IC5.62 (VSS_5); no longer IC1.26 (VSS_2), IC1.41 (VSS_3), IC1.8 (VSS_1)
- net GNDA: now also IC5.73 (AVSS2), IC5.94 (AVSS0), IC5.95 (AVSS1); no longer IC1.48 (AVSS2), IC1.62 (AVSS0), IC1.63 (AVSS1)
- net MTCLKA: now also IC5.58 (P33); no longer IC1.43 (P21)
- net MTCLKB: now also IC5.59 (P32); no longer IC1.44 (P20)
- net MTCLKC: now also IC5.8 (PE4); no longer IC1.64 (P11)
- net MTCLKD: now also IC5.9 (PE3); no longer IC1.42 (P22)
- net MTIOC3B: now also IC5.56 (P71); no longer IC1.38 (P71)
- net MTIOC3D: now also IC5.53 (P74); no longer IC1.35 (P74)
- net MTIOC4A: now also IC5.55 (P72); no longer IC1.37 (P72)
- net MTIOC4B: now also IC5.54 (P73); no longer IC1.36 (P73)
- net MTIOC4C: now also IC5.52 (P75); no longer IC1.34 (P75)
- net MTIOC4D: now also IC5.51 (P76); no longer IC1.33 (P76)
- net MTIOC6B: now also IC5.45 (P95); no longer IC1.27 (P95)
- net MTIOC6D: now also IC5.48 (P92); no longer IC1.30 (P92)
- net MTIOC7A: now also IC5.46 (P94); no longer IC1.28 (P94)
- net MTIOC7B: now also IC5.47 (P93); no longer IC1.29 (P93)
- net MTIOC7C: now also IC5.49 (P91); no longer IC1.31 (P91)
- net MTIOC7D: now also IC5.50 (P90); no longer IC1.32 (P90)
- net PGAVSS0: now also IC5.91 (PH0/PGAVSS0); no longer IC1.59 (PH0/PGAVSS0)
- net PGAVSS1: now also IC5.86 (PH4/PGAVSS1); no longer IC1.55 (PH4/PGAVSS1)
- net TCK: now also IC5.21 (PD4); no longer IC1.15 (PD4)
- net TDI: now also IC5.20 (PD5); no longer IC1.14 (PD5)
- net TDO: now also IC5.22 (PD3); no longer IC1.16 (PD3)
- net TMS: now also IC5.19 (PD6); no longer IC1.13 (PD6)
- net TRST#: now also IC5.18 (PD7); no longer IC1.12 (PD7)
- net VCC: now also C35.1, IC5.14 (VCC_1), IC5.29 (VCC_2), IC5.42 (VCC_3), IC5.60 (VCC_4); no longer IC1.10 (VCC_1), IC1.24 (VCC_2), IC1.40 (VCC_3), R10.1, R11.1, R12.1
- net VDDA: now also IC5.72 (AVCC2), IC5.92 (AVCC1), IC5.93 (AVCC0); no longer IC1.47 (AVCC2), IC1.60 (AVCC1), IC1.61 (AVCC0)
- net at IC1.3 (VCL): no longer C9.1
- net at IC1.7 (P37/XTAL): no longer Y1.3
- net at IC1.9 (P36/EXTAL): no longer Y1.1
- new net: C9.1, IC5.5 (VCL)
- new net: IC5.13 (P36/EXTAL), Y1.1
- new net: IC5.11 (P37/XTAL), Y1.3
- new net AN102: IC5.83 (P46)
- new net AN201: IC5.80 (P53)
- new net AN202: IC5.79 (P54)
- new net AN203: IC5.78 (P55)
- new net AN206: IC5.77 (P60)
- new net AN207: IC5.76 (P61)
- new net AN208: IC5.75 (P62)
- new net AN209: IC5.74 (P63)
- new net AN210/DA0: IC5.71 (P64)
- new net AN211/DA1: IC5.70 (P65)
- new net AN216: IC5.69 (P20)
- new net AN217: IC5.68 (P21)
- new net IRQ4: IC5.7 (P01)
- new net IRQ5: IC5.57 (P70)
- new net MISOA: IC5.24 (PD1)
- new net MOSIA: IC5.23 (PD2)
- new net RSPCKA: IC5.25 (PD0)
- new net SSLA0: IC5.38 (PA3)
- new net SSLA1: IC5.39 (PA2)
- new net SSLA2: IC5.17 (PE0)
- new net SSLA3: IC5.16 (PE1)
Other:
- note added: "TODO： 1. NJM2732のフットプリント修正(SSOP8のフットプリント伸ばす or VSP8にする)…OK 参考：https://akizukidenshi.com/catalog/g/g108891 3. JTAGコネクタ回路ミス修正…OK 4. 耐ESD設計 5. 電荷抜け防止SBD追加…OK 6. IMUのパッドにスルーホールあける 7. PE2(CS)を出力対応ピンに変更する 8. エンコーダSSI化検討…検証済 9. XH⇒PH化, PH⇒PicoBlade化"
- note removed: "TODO： 1. NJM2732のフットプリント修正(SSOP8のフットプリント伸ばす or VSP8にする)…OK 参考：https://akizukidenshi.com/catalog/g/g108891 3. JTAGコネクタ回路ミス修正…OK 4. 耐ESD設計 5. 電荷抜け防止SBD追加…OK 6. IMUのパッドにスルーホールあける 7. PE2(CS)を出力対応ピンに変更する 8. エンコーダSSI化検討 9. XH⇒PH化, PH⇒PicoBlade化"
- moved on the sheet: C1, C10, C2, C6, C7, C8, C9, IC1, R10, R11, R12, Y1

Commit message: ゲートドライバを変更
Parts:
- removed D2: D, Diode_SMD:D_SOD-123, symbol Device:D
- removed IC1: R5F566TEADFM#30, SamacSys_Parts:QFP50P1200X1200X170-64N, symbol SamacSys_Parts:R5F566TEADFM#30
- removed IC3, IC4: DRV8300DPWR, SamacSys_Parts:SOP65P640X120-20N, symbol SamacSys_Parts:DRV8300DPWR
- removed J10: ENC2, Connector_JST:JST_PH_B5B-PH-K_1x05_P2.00mm_Vertical, symbol Connector_Generic:Conn_01x05
- removed J11: ENC2_SPI, Connector_Molex:Molex_PicoBlade_53047-0310_1x03_P1.25mm_Vertical, symbol Connector_Generic:Conn_01x03
- removed J14: FAN, Connector_JST:JST_PH_B2B-PH-K_1x02_P2.00mm_Vertical, symbol Connector_Generic:Conn_01x02
- removed J15: ENC1_SPI, Connector_Molex:Molex_PicoBlade_53047-0310_1x03_P1.25mm_Vertical, symbol Connector_Generic:Conn_01x03
- removed J3: TSL1401, Connector_JST:JST_PH_B5B-PH-K_1x05_P2.00mm_Vertical, symbol Connector_Generic:Conn_01x05
- removed J9: ENC1, Connector_JST:JST_PH_B5B-PH-K_1x05_P2.00mm_Vertical, symbol Connector_Generic:Conn_01x05
- removed R21, R22, R23, R32, R33, R34, R35, R36, R37: 10, Resistor_SMD:R_0603_1608Metric_Pad0.98x0.95mm_HandSolder, symbol Device:R
- added C39: 22u, Capacitor_SMD:C_0805_2012Metric_Pad1.18x1.45mm_HandSolder, symbol Device:C_Small
- added C40: 0.1u, Capacitor_SMD:C_0603_1608Metric_Pad1.08x0.95mm_HandSolder, symbol Device:C_Small
- added C41: 1u, Capacitor_SMD:C_0603_1608Metric_Pad1.08x0.95mm_HandSolder, symbol Device:C_Small
- added C42: 47n, Capacitor_SMD:C_0603_1608Metric_Pad1.08x0.95mm_HandSolder, symbol Device:C_Small
- added C43, C44: 1000p, Capacitor_SMD:C_0603_1608Metric_Pad1.08x0.95mm_HandSolder, symbol Device:C_Small
- added IC3, IC4, IC5: DRV8320HRTVR, SamacSys_Parts:QFN50P500X500X80-33N-D, symbol SamacSys_Parts:DRV8320HRTVR
- added J10, J14: ENC2, Connector_Molex:Molex_PicoBlade_53047-1010_1x10_P1.25mm_Vertical, symbol Connector_Generic:Conn_01x10
- added J11: SENS2, Connector_Molex:Molex_PicoBlade_53047-1010_1x10_P1.25mm_Vertical, symbol Connector_Generic:Conn_01x10
- added J3: SENS1, Connector_Molex:Molex_PicoBlade_53047-1010_1x10_P1.25mm_Vertical, symbol Connector_Generic:Conn_01x10
- added J9: ENC1, Connector_Molex:Molex_PicoBlade_53047-1010_1x10_P1.25mm_Vertical, symbol Connector_Generic:Conn_01x10
- added JP10, JP11, JP12, JP9: JP_or_R, Jumper:SolderJumper-2_P1.3mm_Open_Pad1.0x1.5mm, symbol Jumper:SolderJumper_2_Open
- added Q10, Q11, Q12: FDS6898A, Package_SO:SOIC-8_3.9x4.9mm_P1.27mm, symbol Transistor_FET:FDS6898A
- added R61, R62, R63, R76: 4.7k, Resistor_SMD:R_0603_1608Metric_Pad0.98x0.95mm_HandSolder, symbol Device:R
- added R70, R71, R72, R73: 470, Resistor_SMD:R_0603_1608Metric_Pad0.98x0.95mm_HandSolder, symbol Device:R
- added R74, R75: 0.05/1W, Resistor_SMD:R_2512_6332Metric_Pad1.40x3.35mm_HandSolder, symbol Device:R_US
- C16: value 2.2u -> 47n
- C17, C27: value 2.2u -> 1u
- C20, C26: value 2.2u -> 0.1u
- C24: value 2.2u -> 22u; footprint Capacitor_SMD:C_0603_1608Metric_Pad1.08x0.95mm_HandSolder -> Capacitor_SMD:C_0805_2012Metric_Pad1.18x1.45mm_HandSolder
- C28: value 22u -> 47n; footprint Capacitor_SMD:C_0805_2012Metric_Pad1.18x1.45mm_HandSolder -> Capacitor_SMD:C_0603_1608Metric_Pad1.08x0.95mm_HandSolder
- IC1: renamed from IC5; footprint QFP50P1600X1600X170-100N -> SamacSys_Parts:QFP50P1600X1600X170-100N
- J1: footprint Connector_JST:JST_XH_B2B-XH-A_1x02_P2.50mm_Vertical -> Connector_AMASS:AMASS_XT30U-M_1x02_P5.0mm_Vertical
- J4: value MSENS1 -> MOT3
- J5, J8: footprint Connector_JST:JST_XH_B3B-XH-A_1x03_P2.50mm_Vertical -> Connector_JST:JST_PH_B3B-PH-K_1x03_P2.00mm_Vertical
- J7: value MSENS2 -> ESC
- JP2, JP4: value Jumper -> JP_or_R; footprint Jumper:SolderJumper-2_P1.3mm_Bridged2Bar_Pad1.0x1.5mm -> Jumper:SolderJumper-2_P1.3mm_Open_Pad1.0x1.5mm
- R15, R16, R17: value 10 -> 4.7k
Connections:
- net AN201/IRQ1 is gone; now on net MTIOC9A: J7.2 (Pin_2)
- net MTIOC9C is gone; now on net GTIOC3A: R19.2
- net P64/IRQ8/DA0 is gone; now on net SSLA1: R60.2
- net P65/IRQ9/DA1 is gone; now on net SSLA2: R59.2
- net PB0(CS) is gone; now on net PB4(CS): J13.2 (DAT3/CD), R50.2
- net PB2(CS) is gone; now on net SSLA3: J12.5 (Pin_5), R51.2
- net PE2(CS) is gone; now on net SSLA0: IC2.22 (NCS), R13.2
- net +12V: now also C17.2, C20.2, C24.2, C26.2, C27.2, J7.3 (Pin_3), C39.2, C40.2, C41.2, IC3.3 (VM), IC3.4 (VDRAIN), IC4.3 (VM), IC4.4 (VDRAIN), IC5.3 (VM), IC5.4 (VDRAIN), Q10.7 (D1), Q10.8 (D1), Q11.7 (D1), Q11.8 (D1), Q12.7 (D1), Q12.8 (D1); no longer C28.2
- net AN000: now also C23.1, R25.2, R27.2; no longer R24.2, R26.2
- net AN001: now also C22.1, R24.2, R26.2; no longer R25.2, R27.2
- net AN002: now also C31.1, R41.2, R43.2; no longer C33.1, R2.2, R3.1
- net AN100: now also C44.1, R71.2, R73.2; no longer R40.2, R42.2
- net AN101: now also C43.1, R70.2, R72.2; no longer R41.2, R43.2
- net AN200: now also J11.1 (Pin_1)
- net AN201: now also J11.2 (Pin_2)
- net AN202: now also J11.3 (Pin_3)
- net AN203: now also J11.4 (Pin_4)
- net AN206: now also J11.5 (Pin_5)
- net AN207: now also J11.6 (Pin_6)
- net AN208: now also J11.7 (Pin_7)
- net AN209: now also J11.8 (Pin_8)
- net AN210/DA0: now also J11.9 (Pin_9)
- net AN211/DA1: now also J11.10 (Pin_10)
- net GND: now also C20.1, C24.1, C26.1, J1.1 (Pin_1), J7.1 (Pin_1), C39.1, C40.1, IC3.31 (PGND), IC3.33 (EPAD), IC3.8 (SLA), IC4.31 (PGND), IC4.33 (EPAD), IC4.8 (SLA), IC5.31 (PGND), IC5.33 (EPAD), IC5.8 (SLA), J10.10 (Pin_10), J14.10 (Pin_10), J9.10 (Pin_10), JP10.2 (B), JP11.2 (B), JP12.2 (B), JP9.2 (B), Q12.3 (S2), R74.2, R75.2; no longer C22.2, C23.2, C28.1, C30.2, C31.2, J1.2 (Pin_2)
- net GNDA: now also J3.10 (Pin_10), J3.5 (Pin_5); no longer J4.3 (Pin_3), J7.3 (Pin_3)
- net IRQ4: now also J10.8 (Pin_8), J14.8 (Pin_8)
- net IRQ5: now also J9.8 (Pin_8)
- net MD: now also IC1.6 (MD/FINED)
- net MISOA: now also IC1.36 (PA5), IC2.9 (SDO/AD0), J12.3 (Pin_3), R11.1, J10.3 (Pin_3), J10.9 (Pin_9), J14.3 (Pin_3), J14.9 (Pin_9), J9.3 (Pin_3), J9.9 (Pin_9); no longer IC1.24 (PD1)
- net MOSIA: now also IC1.35 (PB0), IC2.24 (SDA/SDI), J12.2 (Pin_2), R10.1, J10.2 (Pin_2), J14.2 (Pin_2), J9.2 (Pin_2); no longer IC1.23 (PD2)
- net MTCLKA: now also J9.6 (Pin_6)
- net MTCLKB: now also J9.7 (Pin_7)
- net MTCLKC: now also J10.6 (Pin_6), J14.6 (Pin_6)
- net MTCLKD: now also J10.7 (Pin_7), J14.7 (Pin_7)
- net MTIOC0A: now also IC1.61 (P31), J3.9 (Pin_9)
- net MTIOC3B: now also IC3.25 (INHA)
- net MTIOC3D: now also IC3.26 (INLA)
- net MTIOC4A: now also IC3.27 (INHB)
- net MTIOC4B: now also IC3.29 (INHC)
- net MTIOC4C: now also IC3.28 (INLB)
- net MTIOC4D: now also IC3.30 (INLC)
- net MTIOC6B: now also IC4.25 (INHA)
- net MTIOC6D: now also IC4.26 (INLA)
- net MTIOC7A: now also IC4.27 (INHB)
- net MTIOC7B: now also IC4.29 (INHC)
- net MTIOC7C: now also IC4.28 (INLB)
- net MTIOC7D: now also IC4.30 (INLC)
- net PB1/MTIOC0C: now also IC1.34 (PB1), J3.8 (Pin_8)
- net PGAVSS0: now also C22.2, C23.2, C30.2, C31.2, JP2.1 (A), JP10.1 (A), JP9.1 (A)
- net PGAVSS1: now also C43.2, C44.2, JP11.1 (A), JP12.1 (A); no longer JP2.1 (A)
- net RES#: now also IC1.10 (RES#)
- net RSPCKA: now also IC1.32 (PB3), IC2.23 (SCL/SCLK), J12.4 (Pin_4), R12.1, J10.4 (Pin_4), J14.4 (Pin_4), J9.4 (Pin_4); no longer IC1.25 (PD0)
- net SSLA1: now also J9.5 (Pin_5)
- net SSLA2: now also J10.5 (Pin_5), J14.5 (Pin_5), R76.2
- net VCC: now also R10.2, R11.2, R12.2, R15.1, R16.1, R17.1, J10.1 (Pin_1), J14.1 (Pin_1), J9.1 (Pin_1), R61.2, R62.2, R63.2, R76.1
- net VDDA: now also J3.1 (Pin_1), J3.2 (Pin_2), J3.6 (Pin_6); no longer J4.1 (Pin_1), J7.1 (Pin_1)
- net at Q1.3, R4.1: now also J1.2 (Pin_2); no longer J1.1 (Pin_1)
- net Mot.2_SHA: now reaches J8.1 (Pin_1), Q9.1 (S1), Q9.5 (D2), Q9.6 (D2)
- net Mot.2_SHA: now also IC4.6 (SHA); no longer C24.2
- net Mot.2_GHA: now reaches Q9.2 (G1)
- net Mot.2_GHA: now also IC4.5 (GHA)
- net Mot.2_GLA: now reaches Q9.4 (G2)
- net Mot.2_GLA: now also IC4.7 (GLA)
- net Mot.2_SHB: now reaches J8.2 (Pin_2), Q8.1 (S1), Q8.5 (D2), Q8.6 (D2)
- net Mot.2_SHB: now also IC4.11 (SHB); no longer C26.2
- net Mot.2_GHB: now reaches Q8.2 (G1)
- net Mot.2_GHB: now also IC4.12 (GHB)
- net Mot.2_SLB: now reaches Q8.3 (S2), R43.1, R45.1
- net Mot.2_SLB: now also IC4.9 (SLB); no longer C31.1
- net Mot.2_GLB: now reaches Q8.4 (G2)
- net Mot.2_GLB: now also IC4.10 (GLB)
- net Mot.2_SHC: now reaches J8.3 (Pin_3), Q7.1 (S1), Q7.5 (D2), Q7.6 (D2)
- net Mot.2_SHC: now also IC4.14 (SHC); no longer C27.2
- net Mot.2_GHC: now reaches Q7.2 (G1)
- net Mot.2_GHC: now also IC4.13 (GHC)
- net Mot.2_SLC: now reaches Q7.3 (S2), R42.1, R44.1
- net Mot.2_SLC: now also IC4.16 (SLC); no longer C30.1
- net Mot.2_GLC: now reaches Q7.4 (G2)
- net Mot.2_GLC: now also IC4.15 (GLC)
- net Mot.1_GLA: now reaches Q4.4 (G2)
- net Mot.1_GLA: now also IC3.7 (GLA)
- net Mot.1_SHA: now reaches J5.1 (Pin_1), Q4.1 (S1), Q4.5 (D2), Q4.6 (D2)
- net Mot.1_SHA: now also IC3.6 (SHA); no longer C16.2
- net Mot.1_SHB: now reaches J5.2 (Pin_2), Q3.1 (S1), Q3.5 (D2), Q3.6 (D2)
- net Mot.1_SHB: now also IC3.11 (SHB); no longer C17.2
- net Mot.1_GHB: now reaches Q3.2 (G1)
- net Mot.1_GHB: now also IC3.12 (GHB); no longer R16.1
- net Mot.1_SLB: now reaches Q3.3 (S2), R27.1, R30.1
- net Mot.1_SLB: now also IC3.9 (SLB); no longer C23.1
- net Mot.1_GLB: now reaches Q3.4 (G2)
- net Mot.1_GLB: now also IC3.10 (GLB)
- net Mot.1_SHC: now reaches J5.3 (Pin_3), Q2.1 (S1), Q2.5 (D2), Q2.6 (D2)
- net Mot.1_SHC: now also IC3.14 (SHC); no longer C20.2
- net Mot.1_GHC: now reaches Q2.2 (G1)
- net Mot.1_GHC: now also IC3.13 (GHC); no longer R15.1
- net Mot.1_SLC: now reaches Q2.3 (S2), R26.1, R29.1
- net Mot.1_SLC: now also IC3.16 (SLC); no longer C22.1
- net Mot.1_GLC: now reaches Q2.4 (G2)
- net Mot.1_GLC: now also IC3.15 (GLC)
- net Mot.1_GHA: now reaches Q4.2 (G1)
- net Mot.1_GHA: now also IC3.5 (GHA); no longer R17.1
- net at C17.1: now also IC3.2 (VCP)
- net at C16.1: now also IC3.32 (CPL)
- net at C27.1: now also IC4.2 (VCP)
- net at JP3.2 (C), R24.1, R25.1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: now also R70.1, R71.1
- net at C38.1, JP7.1 (A), U1.5 (+): now also J3.7 (Pin_7)
- net GTIOC3A: now reaches IC1.1 (PE5)
- net GTIOC1B: now reaches IC1.26 (PB7)
- net GTIOC1B: now also IC5.28 (INLB)
- net GTIOC2A: now reaches IC1.27 (PB6)
- net GTIOC2A: now also IC5.29 (INHC)
- net GTIOC2B: now reaches IC1.28 (PB5)
- net GTIOC2B: now also IC5.30 (INLC)
- net PB4(CS): now reaches IC1.30 (PB4)
- net MTIOC9A: now reaches IC1.4 (P00)
- net SMOSI12: now reaches IC1.66 (P23)
- net SMOSI12: now also J13.3 (CMD), R61.1
- net SMISO12: now reaches IC1.67 (P22)
- net SMISO12: now also J13.7 (DAT0), R62.1
- net AN103: now reaches IC1.82 (P47)
- net AN103: now also C33.1, R2.2, R3.1
- net AN003: now reaches IC1.87 (P43)
- net AN003: now also C30.1, R40.2, R42.2
- net SCK12: now reaches IC1.96 (P82)
- net SCK12: now also J13.5 (CLK), R63.1
- net AN202/IRQ2 renamed Mot.3_SHB
- net Mot.3_SHB: now also IC5.11 (SHB), Q11.1 (S1), Q11.5 (D2), Q11.6 (D2)
- net AN216 renamed AN216/IRQ7
- net AN216/IRQ7: now also J3.3 (Pin_3)
- net AN217 renamed AN217/IRQ6
- net AN217/IRQ6: now also J3.4 (Pin_4)
- net Mot.1_UH renamed Mot.3_nFAULT
- net Mot.3_nFAULT: now also IC5.17 (NFAULT)
- net Mot.1_VH renamed Mot.2_nFAULT
- net Mot.2_nFAULT: now also IC4.17 (NFAULT)
- net Mot.1_WH renamed Mot.1_nFAULT
- net Mot.1_nFAULT: now also IC3.17 (NFAULT)
- net P00/MTIOC9A: no longer names the net of R28.2
- net P70/IRQ5: no longer names the net of R47.2, SW5.1
- net P96/IRQ4: no longer names the net of R46.2, SW4.1
- removed net SCK11: IC2.23 (SCL/SCLK), J12.4 (Pin_4), J13.5 (CLK), R12.2
- removed net SMISO11: IC2.9 (SDO/AD0), J12.2 (Pin_2), J13.7 (DAT0), R11.2
- removed net SMOSI11: IC2.24 (SDA/SDI), J12.3 (Pin_3), J13.3 (CMD), R10.2
- new net: C16.2, IC3.1 (CPH)
- new net: C42.1, IC5.32 (CPL)
- new net: C42.2, IC5.1 (CPH)
- new net: IC5.18 (MODE), IC5.23 (AGND)
- new net: IC5.19 (IDRIVE), IC5.20 (VDS), IC5.24 (DVDD)
- new net: C41.1, IC5.2 (VCP)
- new net: C28.1, IC4.32 (CPL)
- new net: C28.2, IC4.1 (CPH)
- new net: IC3.18 (MODE), IC3.23 (AGND)
- new net: IC3.19 (IDRIVE), IC3.20 (VDS), IC3.24 (DVDD)
- new net: IC4.18 (MODE), IC4.23 (AGND)
- new net: IC4.19 (IDRIVE), IC4.20 (VDS), IC4.24 (DVDD)
- new net GTIOC0A: IC1.23 (PD2), IC5.25 (INHA)
- new net GTIOC0B: IC1.24 (PD1), IC5.26 (INLA)
- new net GTIOC1A: IC1.25 (PD0), IC5.27 (INHB)
- new net Mot.3_GHA: IC5.5 (GHA), Q12.2 (G1)
- new net Mot.3_GHB: IC5.12 (GHB), Q11.2 (G1)
- new net Mot.3_GHC: IC5.13 (GHC), Q10.2 (G1)
- new net Mot.3_GLA: IC5.7 (GLA), Q12.4 (G2)
- new net Mot.3_GLB: IC5.10 (GLB), Q11.4 (G2)
- new net Mot.3_GLC: IC5.15 (GLC), Q10.4 (G2)
- new net Mot.3_SHA: IC5.6 (SHA), J4.1 (Pin_1), Q12.1 (S1), Q12.5 (D2), Q12.6 (D2)
- new net Mot.3_SHC: IC5.14 (SHC), J4.3 (Pin_3), Q10.1 (S1), Q10.5 (D2), Q10.6 (D2)
- new net Mot.3_SLB: IC5.9 (SLB), Q11.3 (S2), R73.1, R75.1
- new net Mot.3_SLC: IC5.16 (SLC), Q10.3 (S2), R72.1, R74.1
- no-connect marks 7 -> 22
Other:
- note removed: "CPU"
- note removed: "DEBUG I/F"
- note removed: "MOTOR DRIVER"
- note removed: "POWER"
- note removed: "SENSOR"
- note removed: "USER I/F"
- moved on the sheet: BZ1, C1, C10, C11, C12, C13, C14, C15, C16, C17, C18, C19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

Commit message: SPI系配線完了
Parts:
- removed BZ1: Buzzer, Buzzer_Beeper:MagneticBuzzer_Kingstate_KCG0601, symbol Device:Buzzer
- removed C36: 0.1u, Capacitor_SMD:C_0603_1608Metric_Pad1.08x0.95mm_HandSolder, symbol Device:C_Small
- removed J12: LCD, Connector_JST:JST_PH_B6B-PH-K_1x06_P2.00mm_Vertical, symbol Connector_Generic:Conn_01x06
- removed Q5: IRLML6344TRPBF, SamacSys_Parts:SOT95P260X110-3N, symbol SamacSys_Parts:IRLML6344TRPBF
- removed R17, R51: 4.7k, Resistor_SMD:R_0603_1608Metric_Pad0.98x0.95mm_HandSolder, symbol Device:R
- removed R18: 1k, Resistor_SMD:R_0603_1608Metric_Pad0.98x0.95mm_HandSolder, symbol Device:R
- removed R19: 470, Resistor_SMD:R_0603_1608Metric_Pad0.98x0.95mm_HandSolder, symbol Device:R
- removed R20: 100k, Resistor_SMD:R_0603_1608Metric_Pad0.98x0.95mm_HandSolder, symbol Device:R
- J14: value ENC2 -> ENC3
- R52: value 10k -> X1
- R53: value 10k -> X2
Connections:
- net Mot.1_nFAULT is gone; now on net IRQ15: IC3.17 (NFAULT), R15.2
- net Mot.3_nFAULT is gone; now on net IRQ15: IC5.17 (NFAULT)
- net AN200: now also J11.10 (Pin_10); no longer J11.1 (Pin_1)
- net AN201: now also J11.9 (Pin_9); no longer J11.2 (Pin_2)
- net AN202: now also J11.8 (Pin_8); no longer J11.3 (Pin_3)
- net AN203: now also J11.7 (Pin_7); no longer J11.4 (Pin_4)
- net AN206: now also J11.6 (Pin_6); no longer J11.5 (Pin_5)
- net AN207: now also J11.5 (Pin_5); no longer J11.6 (Pin_6)
- net AN208: now also J11.4 (Pin_4); no longer J11.7 (Pin_7)
- net AN209: now also J11.3 (Pin_3); no longer J11.8 (Pin_8)
- net AN210/DA0: now also J11.2 (Pin_2); no longer J11.9 (Pin_9)
- net AN211/DA1: now also J11.1 (Pin_1); no longer J11.10 (Pin_10)
- net GND: now also IC2.25 (T_PAD), R16.2
- net GTIOC3A: now also J14.6 (Pin_6)
- net IRQ4: no longer J14.8 (Pin_8)
- net MTCLKC: no longer J14.6 (Pin_6)
- net MTCLKD: no longer J14.7 (Pin_7)
- net SSLA2: no longer J14.5 (Pin_5), R76.2
- net SSLA3: now also J14.5 (Pin_5), R76.2
- net VCC: no longer R16.1
- net P96(LIGHIT): now reaches R28.2
- net P96(LIGHIT): now also IC1.43 (P96)
- net PB2(GD_EN): now reaches IC5.22 (ENABLE)
- net PB2(GD_EN): now also IC1.33 (PB2), IC3.22 (ENABLE), IC4.22 (ENABLE), R16.1
- net IRQ0: now reaches IC1.100 (P10)
- net IRQ0: now also J14.8 (Pin_8)
- net IRQ15: now reaches IC1.64 (P27)
- net IRQ15: now also IC4.17 (NFAULT)
- net GTIOC3B: now reaches IC1.99 (P11)
- net GTIOC3B: now also J14.7 (Pin_7)
- removed net Mot.2_nFAULT: IC4.17 (NFAULT), R16.2
- no-connect marks 22 -> 15
Other:
- moved on the sheet: C1, C10, C11, C12, C13, C14, C16, C17, C19, C2, C20, C21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

Commit message: ・未配線数０まで完了
Parts:
- removed J7: ESC, Connector_JST:JST_PH_B3B-PH-K_1x03_P2.00mm_Vertical, symbol Connector_Generic:Conn_01x03
- removed JP10, JP11, JP12, JP2, JP4, JP9: JP_or_R, Jumper:SolderJumper-2_P1.3mm_Open_Pad1.0x1.5mm, symbol Jumper:SolderJumper_2_Open
- added R17: 4.7k, Resistor_SMD:R_0603_1608Metric_Pad0.98x0.95mm_HandSolder, symbol Device:R
- renumbered D1 to LED1
Connections:
- net PGAVSS0 is gone; now on net GND: C22.2, C23.2, C30.2, C31.2, IC1.91 (PH0/PGAVSS0)
- net PGAVSS1 is gone; now on net GND: C43.2, C44.2, IC1.86 (PH4/PGAVSS1)
- net GND: now also R17.2
- net GNDA: no longer J3.5 (Pin_5)
- net MTIOC9A: now also J3.5 (Pin_5), R17.1
- net P30: now reaches R47.2, SW5.1
- net P30: now also IC1.63 (P30)
- net P24: now reaches R46.2, SW4.1
- net P24: now also IC1.65 (P24)
- net TXD6: now reaches IC1.97 (P81)
- net RXD6: now reaches IC1.98 (P80)
- no-connect marks 15 -> 9
Other:
- moved on the sheet: C15, J3, R5, R8

Commit message: ・大電流GNDビア修正
Connections:
- net AN102: no longer names the net of IC1.83 (P46)
- net RXD6: no longer names the net of IC1.98 (P80)
- net TDI renamed TDI/RXD1
- net TDO renamed TDO/TXD1
- net TXD6: no longer names the net of IC1.97 (P81)
- no-connect marks 9 -> 12
Other:
- note added: "TODO： 1. NJM2732のフットプリント修正(SSOP8のフットプリント伸ばす or VSP8にする)…OK 参考：https://akizukidenshi.com/catalog/g/g108891 3. JTAGコネクタ回路ミス修正…OK 4. 耐ESD設計 5. 電荷抜け防止SBD追加…OK 6. IMUのパッドにスルーホールあける…OK 8. エンコーダSSI化検討…検証済…OK 9. XH⇒PH化, PH⇒PicoBlade化…OK"
- note removed: "TODO： 1. NJM2732のフットプリント修正(SSOP8のフットプリント伸ばす or VSP8にする)…OK 参考：https://akizukidenshi.com/catalog/g/g108891 3. JTAGコネクタ回路ミス修正…OK 4. 耐ESD設計 5. 電荷抜け防止SBD追加…OK 6. IMUのパッドにスルーホールあける 7. PE2(CS)を出力対応ピンに変更する 8. エンコーダSSI化検討…検証済 9. XH⇒PH化, PH⇒PicoBlade化"
- moved on the sheet: C15
Changed lines of the file:
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@@
 	(generator_version "9.0")
 	(paper "A2")
-	(text "TODO：\n1. NJM2732のフットプリント修正(SSOP8のフットプリント伸ばす or VSP8にする)…OK\n   参考：https://akizukidenshi.com/catalog/g/g108891\n\n3. JTAGコネクタ回路ミス修正…OK\n\n4. 耐ESD設計\n\n5. 電荷抜け防止SBD追加…OK\n\n6. IMUのパッドにスルーホールあける\n\n7. PE2(CS)を出力対応ピンに変更する\n\n8. エンコーダSSI化検討…検証済\n\n9. XH⇒PH化, PH⇒PicoBlade化"
+	(text "TODO：\n1. NJM2732のフットプリント修正(SSOP8のフットプリント伸ばす or VSP8にする)…OK\n   参考：https://akizukidenshi.com/catalog/g/g108891\n\n3. JTAGコネクタ回路ミス修正…OK\n\n4. 耐ESD設計\n\n5. 電荷抜け防止SBD追加…OK\n\n6. IMUのパッドにスルーホールあける…OK\n\n8. エンコーダSSI化検討…検証済…OK\n\n9. XH⇒PH化, PH⇒PicoBlade化…OK"
 		(exclude_from_sim no)
 		(at 10.16 591.82 0)
@@
 	)
 	(no_connect
+		(at 104.14 157.48)
+	)
+	(no_connect
 		(at 100.33 50.8)
 	)
@@
 	)
 	(no_connect
+		(at 104.14 193.04)
+	)
+	(no_connect
+		(at 104.14 195.58)
+	)
+	(no_connect
 		(at 208.28 379.73)
 	)
@@
 	(wire
 		(pts
-			(xy 99.06 281.94) (xy 102.87 281.94)
+			(xy 99.06 279.4) (xy 102.87 279.4)
 		)
 		(stroke
@@
 	(wire
 		(pts
+			(xy 99.06 279.4) (xy 99.06 281.94)
+		)
+		(stroke
+			(width 0)
+			(type default)
+		)
+	)
+	(wire
+		(pts
 			(xy 541.02 114.3) (xy 546.1 114.3)
 		)
@@
 	(wire
 		(pts
-			(xy 99.06 279.4) (xy 99.06 281.94)
-		)
-		(stroke
-			(width 0)
-			(type default)
-		)
-	)
-	(wire
-		(pts
 			(xy 91.44 308.61) (xy 91.44 311.15)
 		)
@@
 	)
 	(image
-		(at 575.31 534.035)
-		(scale 2.27091)
+		(at 711.2 403.225)
+		(scale 4.03592)
 		(data "iVBORw0KGgoAAAANSUhEUgAAApEAAADsCAYAAAAsCP39AAAABHNCSVQICAgIfAhkiAAAIABJREFU"
 			"eJzs3Xd4TNn/wPF3JkWqFCKIsmqURBeCINF79Lr6sqy2hWXxXb0uP21ZRFstoq/FKiF6C1YXmyB6"
@@
 	)
 	(image
-		(at 648.97 327.025)
+		(at 648.97 325.12)
 		(data "iVBORw0KGgoAAAANSUhEUgAABKkAAAK+CAYAAABpQE2nAAAABHNCSVQICAgIfAhkiAAAIABJREFU"
 			"eJzs3Xd4FFUXwOHf7G4KpBBIAUJooXeQ3kvovSkiVUAF6fohoKBYKFKkKAgISBGRTijSW+gdpENI"
@@
 	)
 	(image
-		(at 635 210.185)
+		(at 650.875 190.5)
+		(scale 1.9356)
 		(data "iVBORw0KGgoAAAANSUhEUgAAAowAAAG2CAYAAAD1OteAAAAABHNCSVQICAgIfAhkiAAAIABJREFU"
 			"eJzs3X98U+XdP/5XenpCQzESEIXSpgi7EZEyBRUdRQTnitLhvB3gpzA2boSt7Gai3h3IZOpAhPEd"
@@
 		)
 	)
+	(global_label "TDO{slash}TXD1"
+		(shape input)
+		(at 241.3 38.1 180)
+		(effects
+			(font
+				(size 1.27 1.27)
+				(italic yes)
+			)
+			(justify right)
+		)
+		(property "Intersheetrefs" "${INTERSHEET_REFS}"
+			(at 241.3 38.1 90)
+			(effects
+				(font
+					(size 1.27 1.27)
+				)
+				(hide yes)
+			)
+		)
+	)
 	(global_label "MTIOC7D"
 		(shape output)
@@
 		)
 	)
-	(global_label "TDO"
+	(global_label "TDO{slash}TXD1"
 		(shape output)
 		(at 182.88 208.28 270)
@@
 		)
 	)
+	(global_label "TDI{slash}RXD1"
+		(shape output)
+		(at 241.3 43.18 180)
+		(effects
+			(font
+				(size 1.27 1.27)
+				(italic yes)
+			)
+			(justify right)
+		)
+		(property "Intersheetrefs" "${INTERSHEET_REFS}"
+			(at 241.3 43.18 90)
+			(effects
+				(font
+					(size 1.27 1.27)
+				)
+				(hide yes)
+			)
+		)
+	)
 	(global_label "MTIOC6B"
 		(shape output)
@@
 		)
 	)
-	(global_label "TXD6"
-		(shape output)
-		(at 104.14 193.04 180)
-		(effects
-			(font
-				(size 1.27 1.27)
-				(italic yes)
-			)
-			(justify right)
-		)
-		(property "Intersheetrefs" "${INTERSHEET_REFS}"
-			(at 104.14 193.04 90)
-			(effects
-				(font
-					(size 1.27 1.27)
-				)
-				(hide yes)
-			)
-		)
-	)
 	(global_label "PGAVSS0"
 		(shape output)
@@
 		)
 	)
-	(global_label "RXD6"
-		(shape input)
-		(at 104.14 195.58 180)
-		(effects
-			(font
-				(size 1.27 1.27)
-				(italic yes)
-			)
-			(justify right)
-		)
-		(property "Intersheetrefs" "${INTERSHEET_REFS}"
-			(at 104.14 195.58 90)
-			(effects
-				(font
-					(size 1.27 1.27)
-				)
-				(hide yes)
-			)
-		)
-	)
 	(global_label "SCK12"
 		(shape passive)
@@
 		)
 	)
-	(global_label "TDI"
+	(global_label "TDI{slash}RXD1"
 		(shape input)
 		(at 177.8 208.28 270)
@@
 		)
 	)
-	(global_label "TDO"
-		(shape input)
-		(at 241.3 38.1 180)
-		(effects
-			(font
-				(size 1.27 1.27)
-				(italic yes)
-			)
-			(justify right)
-		)
-		(property "Intersheetrefs" "${INTERSHEET_REFS}"
-			(at 241.3 38.1 0)
-			(effects
-				(font
-					(size 1.27 1.27)
-				)
-				(hide yes)
-			)
-		)
-	)
 	(global_label "Mot.1_SHB"
 		(shape input)
@@
 		)
 	)
-	(global_label "AN102"
-		(shape input)
-		(at 104.14 157.48 180)
-		(effects
-			(font
-				(size 1.27 1.27)
-				(italic yes)
-			)
-			(justify right)
-		)
-		(property "Intersheetrefs" "${INTERSHEET_REFS}"
-			(at 104.14 157.48 90)
-			(effects
-				(font
-					(size 1.27 1.27)
-				)
-				(hide yes)
-			)
-		)
-	)
 	(global_label "AN201"
 		(shape input)
@@
 		)
 	)
-	(global_label "TDI"
-		(shape output)
-		(at 241.3 43.18 180)
-		(effects
-			(font
-				(size 1.27 1.27)
-				(italic yes)
-			)
-			(justify right)
-		)
-		(property "Intersheetrefs" "${INTERSHEET_REFS}"
-			(at 241.3 43.18 0)
-			(effects
-				(font
-					(size 1.27 1.27)
-				)
-				(hide yes)
-			)
-		)
-	)
 	(global_label "P30"
 		(shape input)
@@
 	(symbol
 		(lib_id "Device:C_Small")
-		(at 105.41 281.94 90)
+		(at 105.41 279.4 90)
+		(mirror x)
 		(unit 1)
 		(exclude_from_sim no)
@@
 		(dnp no)
 		(property "Reference" "C15"
-			(at 105.41 278.13 0)
+			(at 105.41 283.21 0)
 			(effects
 				(font
@@
 		)
 		(property "Value" "0.1u"
-			(at 102.87 278.13 0)
+			(at 102.87 283.21 0)
 			(effects
 				(font
@@
 		)
 		(property "Footprint" "Capacitor_SMD:C_0603_1608Metric_Pad1.08x0.95mm_HandSolder"
-			(at 105.41 281.94 0)
+			(at 105.41 279.4 0)
 			(effects
 				(font
@@
 		)
 		(property "Datasheet" "~"
-			(at 105.41 281.94 0)
+			(at 105.41 279.4 0)
 			(effects
 				(font
@@
 		)
 		(property "Description" ""
-			(at 105.41 281.94 0)
+			(at 105.41 279.4 0)
 			(effects
 				(font
@@
 	(symbol
 		(lib_id "power:GNDA")
-		(at 107.95 281.94 90)
+		(at 107.95 279.4 90)
 		(mirror x)
 		(unit 1)
@@
 		(dnp no)
 		(property "Reference" "#PWR030"
-			(at 114.3 281.94 0)
+			(at 114.3 279.4 0)
 			(effects
 				(font
@@
 		)
 		(property "Value" "GNDA"
-			(at 111.76 281.94 0)
+			(at 111.76 279.4 0)
 			(effects
 				(font
@@
 		)
 		(property "Footprint" ""
-			(at 107.95 281.94 0)
+			(at 107.95 279.4 0)
 			(effects
 				(font
@@
 		)
 		(property "Datasheet" ""
-			(at 107.95 281.94 0)
+			(at 107.95 279.4 0)
 			(effects
 				(font
@@
 		)
 		(property "Description" ""
-			(at 107.95 281.94 0)
+			(at 107.95 279.4 0)
 			(effects
 				(font

Commit message: ・初回試作基板の動作を踏まえ，TODO欄に修正箇所を追記． ・PCBアートワーク検討中．
Other:
- note added: "TODO： 4. 耐ESD設計 8. エンコーダSSI化検討…検証済…OK 10. モータ端子汎用化(ピンヘッダ化, レジスト剥き) 11. シャント用ADCピン割変更(S&H機能はANx00~02まで！& 並列変換で高速化) 12. ゲートドライバAGNDをAGNDに接続"
- note added: "参考資料："
- note removed: "TODO： 1. NJM2732のフットプリント修正(SSOP8のフットプリント伸ばす or VSP8にする)…OK 参考：https://akizukidenshi.com/catalog/g/g108891 3. JTAGコネクタ回路ミス修正…OK 4. 耐ESD設計 5. 電荷抜け防止SBD追加…OK 6. IMUのパッドにスルーホールあける…OK 8. エンコーダSSI化検討…検証済…OK 9. XH⇒PH化, PH⇒PicoBlade化…OK"
