File: Tracer_ECU.kicad_sch (KiCad schematic)
At the start: 147 parts, among them IC1 R5F572TFADFP#30, IC2 MPU-6500, IC3 DRV8320HRTVR, IC4 DRV8320HRTVR, IC5 DRV8320HRTVR, J1 BAT, J10 ENC2, J11 SENS2, J13 SDC, J14 ENC3, J2 DBG, J3 SENS1, J4 MOT3, J5 MOT1, J6 LIGHIT, J8 MOT2, J9 ENC1, Q1 TJ8S06M3L(T6L1,NQ), Q10 FDS6898A, Q11 FDS6898A, Q12 FDS6898A, Q2 FDS6898A, Q3 FDS6898A, Q4 FDS6898A, Q6 IRLML6344TRPBF, Q7 FDS6898A, Q8 FDS6898A, Q9 FDS6898A, SW1 SW_SPDT, SW2 SW_Push, SW4 SW_Push, SW5 SW_Push, U1 NJM2732, U2 AZ1117-3.3, Y1 CSTNE20M

Commit message: 初回製造基板(ver.1.0.1)から下記修正． ・シャント用ADCピン割変更．(PGA無しポート割り当てミス修正） ・ゲートドライバAGNDをフローティング→AGNDに接続． ・SBD型番指定，フットプリント変更． ・PchSW FET ピンコンパチ8A→60A品へ変更． ・スナバCをSMD化，多並列化（合計440uF）． ・DRV8320 C_VMを22u→10uF，2012M→1608Mへ変更．（*容量はデータシート準拠） ・DRV8320 Enable回路のプルダウンR削除，ジッタ対策用Cに変更．（*内蔵プルダウンR見落とし） ・汎用AD入力　10入力→8入力へ削減およびTXD/RXD6を追加． ・PCBレイアウト微修正．
Parts:
- removed C3, C34: 220u, Capacitor_THT:CP_Radial_D6.3mm_P2.50mm, symbol Tracer_2.0-rescue:CP1_Small-Device
- removed R16: 4.7k, Resistor_SMD:R_0603_1608Metric_Pad0.98x0.95mm_HandSolder, symbol Device:R
- added C3, C34, C36, C45, C46, C47, C48, C49, C50, C51, C52, C53, C55, C56, C57, C58, C59, C60, C61, C62: 22u, Capacitor_SMD:C_0805_2012Metric_Pad1.18x1.45mm_HandSolder, symbol Tracer_2.0-rescue:CP_Small-Device
- added C54: 0.1u, Capacitor_SMD:C_0603_1608Metric_Pad1.08x0.95mm_HandSolder, symbol Device:C_Small
- C16, C28, C42: value 47n -> 47n/0.1u
- C21, C24, C39: value 22u -> 10u; footprint Capacitor_SMD:C_0805_2012Metric_Pad1.18x1.45mm_HandSolder -> Capacitor_SMD:C_0603_1608Metric_Pad1.08x0.95mm_HandSolder
- C4: value 10u -> 22u
- D3: value D_Schottky -> CUHS20S30; footprint Diode_SMD:D_SOD-123 -> Diode_SMD:D_SOD-323_HandSoldering
- Q1: value TJ8S06M3L(T6L1,NQ) -> TJ60S04M3L
Connections:
- net +12V: now also C3.1, C34.1, C36.1, C45.1, C46.1, C47.1, C48.1, C49.1, C50.1, C51.1, C52.1, C53.1, C55.1, C56.1, C57.1, C58.1, C59.1, C60.1, C61.1, C62.1
- net AN002: now also C44.1, R71.2, R73.2; no longer C31.1, R41.2, R43.2
- net AN100: now also C31.1, R41.2, R43.2; no longer C44.1, R71.2, R73.2
- net AN101: now also C30.1, R40.2, R42.2; no longer C43.1, R70.2, R72.2
- net AN200: no longer J11.10 (Pin_10)
- net AN201: now also C33.1, R2.2, R3.1; no longer J11.9 (Pin_9)
- net GND: now also C3.2, C34.2, C36.2, C45.2, C46.2, C47.2, C48.2, C49.2, C50.2, C51.2, C52.2, C53.2, C54.1, C55.2, C56.2, C57.2, C58.2, C59.2, C60.2, C61.2, C62.2
- net GNDA: now also IC3.18 (MODE), IC3.23 (AGND), IC4.18 (MODE), IC4.23 (AGND), IC5.18 (MODE), IC5.23 (AGND)
- net PB2(GD_EN): now also C54.2
- net AN102: now reaches IC1.83 (P46)
- net AN102: now also C43.1, R70.2, R72.2
- net TXD6: now reaches IC1.97 (P81)
- net TXD6: now also J11.9 (Pin_9)
- net RXD6: now reaches IC1.98 (P80)
- net RXD6: now also J11.10 (Pin_10)
- removed net AN003: C30.1, IC1.87 (P43), R40.2, R42.2
- removed net AN103: C33.1, IC1.82 (P47), R2.2, R3.1
- no-connect marks 12 -> 11
Other:
- note added: "TODO： 4. 耐ESD設計 8. エンコーダSSI化検討…検証済…OK 10. モータ端子汎用化(ピンヘッダ化, レジスト剥き) 11. シャント用ADCピン割変更(S&H機能はANx00~02まで！& 並列変換で高速化) 12. ゲートドライバAGNDをAGNDに接続…OK 13. SBDフットプリント変更…OK 14. PchSW FET ピンコンパチ8A→60A品変更…OK 15. スナバC SMD&多並列化…OK 16. DRV8320 Cvm_2 22u→10uF 2012M→1608M, その他周辺回路改善…OK"
- note removed: "TODO： 4. 耐ESD設計 8. エンコーダSSI化検討…検証済…OK 10. モータ端子汎用化(ピンヘッダ化, レジスト剥き) 11. シャント用ADCピン割変更(S&H機能はANx00~02まで！& 並列変換で高速化) 12. ゲートドライバAGNDをAGNDに接続"
- moved on the sheet: C1, C10, C2, C32, C35, C4, C5, C6, C7, C8, C9, D3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

Commit message: 回路修正完了(2相/3相選択版) 小型化のため最小ビア径0.45mm/最小配線幅0.2mmへ変更 レイアウト修正8割方完了．一旦コミット
Parts:
- added JP2, JP4: Jumper, Jumper:SolderJumper-3_P1.3mm_Open_RoundedPad1.0x1.5mm, symbol Jumper:SolderJumper_3_Open
- added LED2: LED, LED_SMD:LED_0603_1608Metric_Pad1.05x0.95mm_HandSolder, symbol Device:LED
- added R16, R18: 0.05/1W, Resistor_SMD:R_2512_6332Metric_Pad1.40x3.35mm_HandSolder, symbol Device:R_US
- added R19, R20, R21: 47k, Resistor_SMD:R_0603_1608Metric_Pad0.98x0.95mm_HandSolder, symbol Device:R
- R24, R25, R26, R27, R40, R41, R42, R43, R70, R71, R72, R73: value 470 -> 470F
- R38, R39: value 10k -> 10kF
- R52: value X1 -> XF
- R53: value X2 -> XF
Connections:
- net GND: now also R16.2, R18.2; no longer IC3.8 (SLA), IC4.8 (SLA), Q4.3 (S2), Q9.3 (S2)
- net GNDA: now also R19.2, R20.2, R21.2; no longer IC3.18 (MODE), IC4.18 (MODE), IC5.18 (MODE)
- net IRQ15: now also LED2.1 (K); no longer R15.2
- net Mot.3_SLB: now also JP2.1 (A); no longer R73.1
- net Mot.3_SLC: now also JP4.1 (A); no longer R72.1
- new net: IC5.18 (MODE), R21.1
- new net: LED2.2 (A), R15.2
- new net: JP4.2 (C), R72.1
- new net: IC4.18 (MODE), R20.1
- new net: JP2.2 (C), R73.1
- new net: IC3.18 (MODE), R19.1
- new net M1_RU+: IC3.8 (SLA), JP2.3 (B), Q4.3 (S2), R16.1
- new net M2_RU+: IC4.8 (SLA), JP4.3 (B), Q9.3 (S2), R18.1
Other:
- note added: "TODO： 4. 耐ESD設計 8. エンコーダSSI化検討…検証済…OK 10. JTAGリボンコネクタ化検討 11. シャント用ADCピン割変更(S&H機能はANx00~02まで！& 並列変換で高速化)…OK 12. ゲートドライバAGNDをAGNDに接続…OK 13. SBDフットプリント変更…OK 14. PchSW FET ピンコンパチ8A→60A品変更…OK 15. スナバC SMD&多並列化…OK 16. DRV8320 Cvm_2 22u→10uF 2012M→1608M, その他周辺回路改善…OK 17.一部を集合抵抗化"
- note removed: "TODO： 4. 耐ESD設計 8. エンコーダSSI化検討…検証済…OK 10. モータ端子汎用化(ピンヘッダ化, レジスト剥き) 11. シャント用ADCピン割変更(S&H機能はANx00~02まで！& 並列変換で高速化) 12. ゲートドライバAGNDをAGNDに接続…OK 13. SBDフットプリント変更…OK 14. PchSW FET ピンコンパチ8A→60A品変更…OK 15. スナバC SMD&多並列化…OK 16. DRV8320 Cvm_2 22u→10uF 2012M→1608M, その他周辺回路改善…OK"
- moved on the sheet: C43, C44, R15, R70, R71, R72, R73, R74, R75
